File: pcb/d1led.kicad_pcb (KiCad board)
At the start: 2 copper layers, 25.4 x 25.4 mm, 16 parts, among them U1 WeMos_D1_mini

Commit message: Add files via upload
Connections:
- U1 pad 11: Net-(U1-Pad11) -> DIN
- U1 pad 3: DIN -> Net-(U1-Pad3)
Routing:
- net DIN: track 6.59 -> 28.0 mm, vias 0 -> 3
Other:
- board text added: "D1 mini LED shield v0.1.4"
- board text removed: "D1 mini LED shield v0.1.3"
